File: MCU_ESP32-C6.kicad_sch (KiCad schematic)
At the start: 33 parts, among them J2 Conn_01x12, J3 Conn_01x12, SW1 SW_Push, SW2 SW_Push, U1 ESP32-C6, U2 W25Q16JVSSIQ

Commit message: -add fuse -change connectors footprint - push button footprint changed
Parts:
- E1: footprint AMCA31-2R450G-S1F-T3:XDCR_AMCA31-2R450G-S1F-T3 -> 1_ESP32:XDCR_AMCA31-2R450G-S1F-T3
- J2: footprint Connector_PinSocket_2.00mm:PinSocket_1x12_P2.00mm_Vertical_SMD_Pin1Left -> Connector_PinSocket_2.54mm:PinSocket_1x12_P2.54mm_Vertical
- J3: footprint Connector_PinSocket_2.00mm:PinSocket_1x12_P2.00mm_Vertical_SMD_Pin1Right -> Connector_PinSocket_2.54mm:PinSocket_1x12_P2.54mm_Vertical
- SW1, SW2: footprint (none) -> 1_ESP32:SW4_PTS815 SJM 250 SMTR LFS_CNK
Changed lines of the file:
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@@
 			)
 		)
-		(property "Footprint" ""
+		(property "Footprint" "1_ESP32:SW4_PTS815 SJM 250 SMTR LFS_CNK"
 			(at 176.53 83.82 0)
 			(effects
@@
 			)
 		)
-		(property "Footprint" "Connector_PinSocket_2.00mm:PinSocket_1x12_P2.00mm_Vertical_SMD_Pin1Left"
+		(property "Footprint" "Connector_PinSocket_2.54mm:PinSocket_1x12_P2.54mm_Vertical"
 			(at 262.89 85.09 0)
 			(effects
@@
 			)
 		)
-		(property "Footprint" "AMCA31-2R450G-S1F-T3:XDCR_AMCA31-2R450G-S1F-T3"
+		(property "Footprint" "1_ESP32:XDCR_AMCA31-2R450G-S1F-T3"
 			(at 181.61 127 0)
 			(effects
@@
 			)
 		)
-		(property "Footprint" "Connector_PinSocket_2.00mm:PinSocket_1x12_P2.00mm_Vertical_SMD_Pin1Right"
+		(property "Footprint" "Connector_PinSocket_2.54mm:PinSocket_1x12_P2.54mm_Vertical"
 			(at 240.03 85.09 0)
 			(effects
@@
 			)
 		)
-		(property "Footprint" ""
+		(property "Footprint" "1_ESP32:SW4_PTS815 SJM 250 SMTR LFS_CNK"
 			(at 50.8 81.28 0)
 			(effects
